Commit message: fixed the code to train with d4pg agents

File: urdf/turtlebot3_burger.urdf.xacro (robot description, xacro)
@@ -50,8 +50,16 @@
         <cylinder length="0.018" radius="0.033"/>
       </geometry>
+      <surface>
+        <friction>
+          <ode>
+            <mu>2</mu>
+            <mu2>2</mu2>
+          </ode>
+        </friction>
+      </surface>
     </collision>
     <inertial>
       <origin xyz="0 0 0" />
-      <mass value="2.8498940e-02" />
+      <mass value="1" />
       <inertia ixx="1.1175580e-05" ixy="-4.2369783e-11" ixz="-5.9381719e-09"
                iyy="1.1192413e-05" iyz="-1.4400107e-11"
@@ -78,8 +86,16 @@
         <cylinder length="0.018" radius="0.033"/>
       </geometry>
+      <surface>
+        <friction>
+          <ode>
+            <mu>2</mu>
+            <mu2>2</mu2>
+          </ode>
+        </friction>
+      </surface>
     </collision>
     <inertial>
       <origin xyz="0 0 0" />
-      <mass value="2.8498940e-02" />
+      <mass value="1" />
       <inertia ixx="1.1175580e-05" ixy="-4.2369783e-11" ixz="-5.9381719e-09"
                iyy="1.1192413e-05" iyz="-1.4400107e-11"
