Commit message: added jackel robot

File: urdf/turtlebot3_burger.gazebo.xacro (robot description, xacro)
@@ -12,5 +12,5 @@
     <kd>10.0</kd>
     <minDepth>0.001</minDepth>
-    <maxVel>0.1</maxVel>
+    <maxVel>1</maxVel>
     <fdir1>1 0 0</fdir1>
     <material>Gazebo/FlatBlack</material>
@@ -22,5 +22,5 @@
     <kd>10.0</kd>
     <minDepth>0.001</minDepth>
-    <maxVel>0.1</maxVel>
+    <maxVel>1</maxVel>
     <fdir1>1 0 0</fdir1>
     <material>Gazebo/FlatBlack</material>

File: urdf/turtlebot3_burger.urdf.xacro (robot description, xacro)
@@ -117,5 +117,5 @@
     <inertial>
       <origin xyz="0 0 0" />
-      <mass value="0.005" />
+      <mass value="0.01" />
       <inertia ixx="0.001" ixy="0.0" ixz="0.0"
                iyy="0.001" iyz="0.0"
@@ -149,5 +149,5 @@
     </collision>
     <inertial>
-      <mass value="0.114" />
+      <mass value="0.514" />
       <origin xyz="0 0 0" />
       <inertia ixx="0.001" ixy="0.0" ixz="0.0"
